File: stegosaurus-schema/stegosaurus-schema.kicad_sch (KiCad schematic)
At the start: 13 parts, among them J1 DIN-5_180degree, J2 DIN-5_180degree, J3 Screw_Terminal_01x06, J4 Barrel_Jack_MountingPin, U1 6N138, U2 LM7805_TO220

Commit message: schematics
Connections:
- net GND: now also J4.1; no longer J4.2
- net at C1.1, J3.6 (Pin_6), U2.1 (VI): now also J4.2; no longer J4.1
Other:
- note added: "3.3V is an input 5V is an output VIN can be either (must be > 7V) GND is shared"
- note removed: "3.3V is an input 5V is an output VIN probably not used"
- moved on the sheet: J4
Changed lines of the file:
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@@
 	)
 	(no_connect
-		(at 34.29 44.45)
+		(at 34.29 39.37)
 	)
 	(no_connect
@@
 	(wire
 		(pts
+			(xy 41.91 34.29) (xy 57.15 34.29)
+		)
+		(stroke
+			(width 0)
+			(type default)
+		)
+	)
+	(wire
+		(pts
 			(xy 224.79 60.96) (xy 223.52 60.96)
 		)
@@
 	(wire
 		(pts
-			(xy 41.91 34.29) (xy 57.15 34.29)
-		)
-		(stroke
-			(width 0)
-			(type default)
-		)
-	)
-	(wire
-		(pts
 			(xy 148.59 34.29) (xy 215.9 34.29)
 		)
@@
 	(wire
 		(pts
-			(xy 41.91 39.37) (xy 44.45 39.37)
-		)
-		(stroke
-			(width 0)
-			(type default)
-		)
-	)
-	(wire
-		(pts
 			(xy 68.58 41.91) (xy 68.58 45.72)
 		)
@@
 	(wire
 		(pts
+			(xy 44.45 29.21) (xy 41.91 29.21)
+		)
+		(stroke
+			(width 0)
+			(type default)
+		)
+	)
+	(wire
+		(pts
 			(xy 57.15 34.29) (xy 60.96 34.29)
 		)
@@
 	(wire
 		(pts
-			(xy 44.45 39.37) (xy 44.45 45.72)
+			(xy 44.45 29.21) (xy 44.45 40.64)
 		)
 		(stroke
@@
 		)
 	)
-	(text "3.3V is an input\n5V is an output\nVIN probably not used"
-		(exclude_from_sim no)
-		(at 251.968 63.5 0)
+	(text "3.3V is an input\n5V is an output\nVIN can be either (must be > 7V)\nGND is shared"
+		(exclude_from_sim no)
+		(at 241.046 61.976 0)
 		(effects
 			(font
 				(size 1.27 1.27)
 			)
+			(justify left)
 		)
 	)
@@
 	(text "9V"
 		(exclude_from_sim no)
-		(at 25.908 36.83 0)
+		(at 25.908 31.75 0)
 		(effects
 			(font
@@
 	(symbol
 		(lib_id "Connector:Barrel_Jack_MountingPin")
-		(at 34.29 36.83 0)
+		(at 34.29 31.75 0)
 		(unit 1)
 		(exclude_from_sim no)
@@
 		(fields_autoplaced yes)
 		(property "Reference" "J4"
-			(at 34.29 27.94 0)
+			(at 34.29 22.86 0)
 			(effects
 				(font
@@
 		)
 		(property "Value" "Barrel_Jack_MountingPin"
-			(at 34.29 30.48 0)
+			(at 34.29 25.4 0)
 			(effects
 				(font
@@
 		)
 		(property "Footprint" "Connector_BarrelJack:BarrelJack_CUI_PJ-102AH_Horizontal"
-			(at 35.56 37.846 0)
+			(at 35.56 32.766 0)
 			(effects
 				(font
@@
 		)
 		(property "Datasheet" "~"
-			(at 35.56 37.846 0)
+			(at 35.56 32.766 0)
 			(effects
 				(font
@@
 		)
 		(property "Description" "DC Barrel Jack with a mounting pin"
-			(at 34.29 36.83 0)
+			(at 34.29 31.75 0)
 			(effects
 				(font
@@
 	(symbol
 		(lib_id "power:GNDREF")
-		(at 44.45 45.72 0)
+		(at 44.45 40.64 0)
 		(unit 1)
 		(exclude_from_sim no)
@@
 		(fields_autoplaced yes)
 		(property "Reference" "#PWR08"
-			(at 44.45 52.07 0)
+			(at 44.45 46.99 0)
 			(effects
 				(font
@@
 		)
 		(property "Value" "GND"
-			(at 44.45 50.8 0)
+			(at 44.45 45.72 0)
 			(effects
 				(font
@@
 		)
 		(property "Footprint" ""
-			(at 44.45 45.72 0)
+			(at 44.45 40.64 0)
 			(effects
 				(font
@@
 		)
 		(property "Datasheet" ""
-			(at 44.45 45.72 0)
+			(at 44.45 40.64 0)
 			(effects
 				(font
@@
 		)
 		(property "Description" "Power symbol creates a global label with name \"GNDREF\" , reference supply ground"
-			(at 44.45 45.72 0)
-			(effects
-				(font
+			(at 44.45 40.64 0)
+			(effects
+				(font

Commit message: more values
Connections:
- net +3.3V: now also J3.3 (Pin_3); no longer J3.4 (Pin_4)
- net GND: now also J3.4 (Pin_4); no longer J3.3 (Pin_3)
- net at C1.1, J4.2, U2.1 (VI): now also J3.1 (Pin_1); no longer J3.6 (Pin_6)
- net at R2.2, U1.6 (VO2): now also J3.6 (Pin_6); no longer J3.1 (Pin_1)
- net at C2.1, U1.8 (VCC), U2.3 (VO): now also J3.2 (Pin_2); no longer J3.5 (Pin_5)
- net at R3.1: now also J2.5; no longer J3.2 (Pin_2)
- net at R3.2: now also J3.5 (Pin_5); no longer J2.5
Other:
- moved on the sheet: C1, C2, J2, J3, J4, R2, R3, R4, U2
